File: ATU_0.sch (KiCad schematic (older format))
At the start: 46 parts, among them J1 Screw_Terminal_01x02, J2 HC06_Module, J3 Barrel_Jack_Switch, J4 Screw_Terminal_01x02, J5 Conn_01x15, J6 Conn_02x04_Odd_Even, J7 Conn_01x05, U2 TPIC6C596

Commit message: new commit
Parts:
- R3: value R -> 820R
Other:
- note added: "Inputs of TPIC6C596 are 5V-CMOS-compatible, but not TTL-compatible.\nThis is OK for the Arduino Nano, but for the connection to 3.3V-IOs a level converter will be required!"
- note added: "for future expansion"
- moved on the sheet: D1, D2, J3, NT2, R1, R3, RL1, RL2, TP1, TP2, TP3, TP4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
