File: Csektion.sch (KiCad schematic (older format))
At the start: 56 parts, among them U5 TPIC6C596, U6 TPIC6C596

Commit message: new commit
Changed lines of the file:
@@
 encoding utf-8
 Sheet 3 3
-Title ""
-Date ""
-Rev ""
-Comp ""
-Comment1 ""
+Title "ATU_0"
+Date "2019-11-03"
+Rev "1"
+Comp "DM1CR (Christian Rausch aka papamidas)"
+Comment1 "HF Antenna Tuner"
 Comment2 ""
 Comment3 ""
@@
 $EndComp
 Wire Wire Line
-	3200 2150 3200 2200
-Wire Wire Line
-	3200 2200 1550 2200
-Wire Wire Line
-	1550 2200 1550 3200
+	3200 2150 3200 2250
+Wire Wire Line
+	3200 2250 1550 2250
+Wire Wire Line
+	1550 2250 1550 3200
 Wire Wire Line
 	1550 3200 1700 3200
@@
 	2300 3200 2450 3200
 Wire Wire Line
-	2450 3200 2450 2250
-Wire Wire Line
-	2450 2250 3300 2250
-Wire Wire Line
-	3300 2250 3300 2150
-Wire Wire Line
-	2550 3200 2550 2300
-Wire Wire Line
-	3400 2300 3400 2150
+	2450 3200 2450 2350
+Wire Wire Line
+	2450 2350 3300 2350
+Wire Wire Line
+	3300 2350 3300 2150
+Wire Wire Line
+	2550 3200 2550 2450
+Wire Wire Line
+	3400 2450 3400 2150
 Wire Wire Line
 	3400 3200 3500 3200
@@
 	4450 3200 4550 3200
 Wire Wire Line
-	4550 3200 4550 2300
-Wire Wire Line
-	4550 2300 3700 2300
-Wire Wire Line
-	3700 2300 3700 2150
+	4550 3200 4550 2450
+Wire Wire Line
+	4550 2450 3700 2450
+Wire Wire Line
+	3700 2450 3700 2150
 Wire Wire Line
 	4950 3200 4650 3200
 Wire Wire Line
-	4650 3200 4650 2250
-Wire Wire Line
-	4650 2250 3800 2250
-Wire Wire Line
-	3800 2250 3800 2150
+	4650 3200 4650 2350
+Wire Wire Line
+	4650 2350 3800 2350
+Wire Wire Line
+	3800 2350 3800 2150
 Wire Wire Line
 	5550 3200 5700 3200
 Wire Wire Line
-	5700 3200 5700 2200
-Wire Wire Line
-	5700 2200 3900 2200
-Wire Wire Line
-	3900 2200 3900 2150
-Wire Wire Line
-	2550 2300 3400 2300
+	5700 3200 5700 2250
+Wire Wire Line
+	5700 2250 3900 2250
+Wire Wire Line
+	3900 2250 3900 2150
+Wire Wire Line
+	2550 2450 3400 2450
 Wire Wire Line
 	2550 3200 2800 3200
@@
 $EndComp
 Wire Wire Line
-	7500 2150 7500 2200
-Wire Wire Line
-	7500 2200 5850 2200
-Wire Wire Line
-	5850 2200 5850 3200
+	7500 2150 7500 2250
+Wire Wire Line
+	7500 2250 5850 2250
+Wire Wire Line
+	5850 2250 5850 3200
 Wire Wire Line
 	5850 3200 6000 3200
@@
 	6600 3200 6750 3200
 Wire Wire Line
-	6750 3200 6750 2250
-Wire Wire Line
-	7600 2250 7600 2150
-Wire Wire Line
-	6850 3200 6850 2300
+	6750 3200 6750 2350
+Wire Wire Line
+	7600 2350 7600 2150
+Wire Wire Line
+	6850 3200 6850 2450
 Wire Wire Line
 	7700 3200 7800 3200
@@
 	8750 3200 8850 3200
 Wire Wire Line
-	8850 3200 8850 2300
-Wire Wire Line
-	8850 2300 8000 2300
-Wire Wire Line
-	8000 2300 8000 2150
+	8850 3200 8850 2450
+Wire Wire Line
+	8850 2450 8000 2450
+Wire Wire Line
+	8000 2450 8000 2150
 Wire Wire Line
 	9250 3200 8950 3200
 Wire Wire Line
-	8950 3200 8950 2250
-Wire Wire Line
-	8950 2250 8100 2250
-Wire Wire Line
-	8100 2250 8100 2150
+	8950 3200 8950 2350
+Wire Wire Line
+	8950 2350 8100 2350
+Wire Wire Line
+	8100 2350 8100 2150
 Wire Wire Line
 	9850 3200 10000 3200
 Wire Wire Line
-	10000 3200 10000 2200
-Wire Wire Line
-	10000 2200 8200 2200
-Wire Wire Line
-	8200 2200 8200 2150
-Wire Wire Line
-	6850 2300 7700 2300
+	10000 3200 10000 2250
+Wire Wire Line
+	10000 2250 8200 2250
+Wire Wire Line
+	8200 2250 8200 2150
+Wire Wire Line
+	6850 2450 7700 2450
 Wire Wire Line
 	6850 3200 7100 3200
@@
 $EndComp
 Wire Wire Line
-	4000 2150 6000 2150
-Wire Wire Line
-	6000 2150 6000 1150
-Wire Wire Line
-	6000 1150 7700 1150
-Wire Wire Line
-	7700 1150 7700 1250
+	4000 2150 5800 2150
+Wire Wire Line
+	5800 2150 5800 1200
+Wire Wire Line
+	5800 1200 7700 1200
+Wire Wire Line
+	7700 1200 7700 1250
 Wire Wire Line
 	3600 1250 3600 1200
 Wire Wire Line
-	3600 1050 7900 1050
-Wire Wire Line
-	7900 1050 7900 1250
+	3600 1100 7900 1100
+Wire Wire Line
+	7900 1100 7900 1250
 Wire Wire Line
 	7800 1250 7800 1000
@@
 	3300 1250 3300 900
 Wire Wire Line
-	3300 850  7600 850
-Wire Wire Line
-	7600 850  7600 1250
+	3300 900  7600 900
+Wire Wire Line
+	7600 900  7600 1250
 Wire Wire Line
 	7500 1250 7500 800
@@
 	2550 900  3300 900
 Connection ~ 3300 900
-Wire Wire Line
-	3300 900  3300 850
 Text HLabel 2550 1000 0    50   Input ~ 0
 SERIN
@@
 Connection ~ 3600 1200
 Wire Wire Line
-	3600 1200 3600 1050
+	3600 1200 3600 1100
 Text HLabel 2550 1200 0    50   Input ~ 0
 nSRCLR
@@
 $EndComp
 Wire Wire Line
-	6750 2250 7600 2250
-Wire Wire Line
-	7700 2300 7700 2150
+	6750 2350 7600 2350
+Wire Wire Line
+	7700 2450 7700 2150
 $Comp
 L ATU_0-rescue:TPIC6C596-tpic6c596 U?
@@
 $EndComp
 Wire Wire Line
-	2300 3600 2450 3600
-Wire Wire Line
-	2450 3600 2450 4200
-Wire Wire Line
-	2450 4200 2300 4200
+	2300 3600 2500 3600
+Wire Wire Line
+	2500 3600 2500 4200
+Wire Wire Line
+	2500 4200 2300 4200
 Wire Wire Line
 	9850 4200 10050 4200
